File: pcb/cpu.sch (KiCad schematic (older format))
At the start: 5 parts, among them J100 Conn_02x05_Odd_Even

Commit message: sch: working on system config
Parts:
- removed D100: 1N5819, Diode_SMD:D_SOD-123, symbol Device:D_Schottky
- removed J100: Conn_02x05_Odd_Even, Connector_PinHeader_1.27mm:PinHeader_2x05_P1.27mm_Vertical_SMD, symbol Connector_Generic:Conn_02x05_Odd_Even
- removed R108: 10K, Resistor_SMD:R_0603_1608Metric, symbol Device:R
- added C107, C108, C110, C117, C118: 470nF, Capacitor_SMD:C_0402_1005Metric, symbol Device:C
- added C109, C119: 4.7uF, Capacitor_SMD:C_0603_1608Metric, symbol Device:C
- added FPGA_JTAG1: Conn_02x05_Odd_Even, Connector_PinHeader_1.27mm:PinHeader_2x05_P1.27mm_Vertical_SMD, symbol Connector_Generic:Conn_02x05_Odd_Even
- added R101, R? (x10): 20K, Capacitor_SMD:C_0402_1005Metric, symbol Device:R
- added R102: DNP, Capacitor_SMD:C_0402_1005Metric, symbol Device:R
- added R103, R105: 10K, Capacitor_SMD:C_0402_1005Metric, symbol Device:R
- added R104: 33R, Capacitor_SMD:C_0402_1005Metric, symbol Device:R
- added R117, R? (x5): 4.7K, Capacitor_SMD:C_0402_1005Metric, symbol Device:R
- added R?: 330, Capacitor_SMD:C_0402_1005Metric, symbol Device:R
- added R?: 0, Capacitor_SMD:C_0402_1005Metric, symbol Device:R
- added U? (x2): XC7Z007S-CLG400, symbol symbols:XC7Z007S-CLG400
- added X100: 33.33MHz, Oscillator:Oscillator_SMD_Abracon_ASE-4Pin_3.2x2.5mm, symbol Oscillator:ASE-xxxMHz
Connections:
- net labels added: +1V8, FPGA_DONE, FPGA_INIT_B, FPGA_TCK, FPGA_TDI, FPGA_TDO, FPGA_TMS, MODE0, MODE1, MODE2, MODE3, MODE4, NAND_ALE, NAND_BUSY, NAND_CE_B, NAND_CLE, NAND_IO0, NAND_IO1, NAND_IO2, NAND_IO3, NAND_IO4, NAND_IO5, NAND_IO6, NAND_IO7, NAND_RE_B, NAND_WE_B, PS_CLK, PS_POR_B, USB_RESET_B, VMODE0, VMODE1
- net labels removed: MPU_JTAG_TCK, MPU_JTAG_TDO, MPU_JTAG_TMS, POR
- wire segments 17 -> 131
- no-connect marks 3 -> 9
Other:
- note added: "MODE0: \nHIGH-SD card\nLOW-NAND"
- note added: "MODE3:\nHIGH-Indep JTAG\nLOW-Cascade JTAG"
- note removed: "JTAG"
- moved on the sheet: D101, R100
