File: pcb/lcd.sch (KiCad schematic (older format))
At the start: 0 parts

Commit message: sch: working on system config
Parts:
- added C501, C509: 22uF/35V, Capacitor_SMD:C_1206_3216Metric, symbol Device:C
- added C508: 10uF, Capacitor_SMD:C_0603_1608Metric, symbol Device:C
- added C512: 4.7uF/35V, Capacitor_SMD:C_0603_1608Metric, symbol Device:C
- added C? (x6): 100nF, Capacitor_SMD:C_0402_1005Metric, symbol Device:C
- added C?: 220pF, Capacitor_SMD:C_0603_1608Metric, symbol Device:C
- added D501: MBR0530, Diode_SMD:D_SOD-123, symbol Device:D_Schottky
- added J? (x3): Conn_01x15, symbol Connector_Generic:Conn_01x15
- added L500: 47uH, Inductor_SMD:L_Vishay_IHLP-1212, symbol Device:L
- added R501: 10K, Resistor_SMD:R_0603_1608Metric, symbol Device:R
- added R503: 330K/1%, Resistor_SMD:R_0603_1608Metric, symbol Device:R
- added R509: 22K/1%, Resistor_SMD:R_0603_1608Metric, symbol Device:R
- added RV500: 100K, footprints:Potentiometer_RK14J, symbol Device:R_POT
- added U?: LT1615, Package_TO_SOT_SMD:TSOT-23-5, symbol symbols:LT1615
Connections:
- new net: R503.1, RV500.1
- new net: C?.1, R509.1, RV500.2, RV500.3, U?.3 (NFB)
- new net: D501.2 (A), L500.2, U?.1 (SW)
- new net +3V3: C508.1, C?.1, C?.1, C?.1, J?.5 (Pin_5), J?.5 (Pin_5), J?.5 (Pin_5), L500.1, U?.5 (VIN)
- new net GND: C501.2, C508.2, C509.2, C512.1, C?.2, C?.2, C?.2, C?.2, C?.2, C?.2, J?.6 (Pin_6), J?.6 (Pin_6), J?.6 (Pin_6), R501.2, R509.2, U?.2 (GND)
- new net LCD1_DL0: J?.12 (Pin_12)
- new net LCD1_DL1: J?.13 (Pin_13)
- new net LCD1_DL2: J?.14 (Pin_14)
- new net LCD1_DL3: J?.15 (Pin_15)
- new net LCD1_DU0: J?.8 (Pin_8)
- new net LCD1_DU1: J?.9 (Pin_9)
- new net LCD1_DU2: J?.10 (Pin_10)
- new net LCD1_DU3: J?.11 (Pin_11)
- new net LCD2_DL0: J?.12 (Pin_12)
- new net LCD2_DL1: J?.13 (Pin_13)
- new net LCD2_DL2: J?.14 (Pin_14)
- new net LCD2_DL3: J?.15 (Pin_15)
- new net LCD2_DU0: J?.8 (Pin_8)
- new net LCD2_DU1: J?.9 (Pin_9)
- new net LCD2_DU2: J?.10 (Pin_10)
- new net LCD2_DU3: J?.11 (Pin_11)
- new net LCD3_DL0: J?.12 (Pin_12)
- new net LCD3_DL1: J?.13 (Pin_13)
- new net LCD3_DL2: J?.14 (Pin_14)
- new net LCD3_DL3: J?.15 (Pin_15)
- new net LCD3_DU0: J?.8 (Pin_8)
- new net LCD3_DU1: J?.9 (Pin_9)
- new net LCD3_DU2: J?.10 (Pin_10)
- new net LCD3_DU3: J?.11 (Pin_11)
- new net LCD_CP: J?.3 (Pin_3), J?.3 (Pin_3), J?.3 (Pin_3)
- new net LCD_DISPOFF: J?.4 (Pin_4), J?.4 (Pin_4), J?.4 (Pin_4)
- new net LCD_FLM: J?.1 (Pin_1), J?.1 (Pin_1), J?.1 (Pin_1)
- new net LCD_LP: J?.2 (Pin_2), J?.2 (Pin_2), J?.2 (Pin_2)
- new net VEE: C501.1, C509.1, C512.2, C?.1, C?.1, C?.1, C?.2, D501.1 (K), J?.7 (Pin_7), J?.7 (Pin_7), J?.7 (Pin_7), R503.2
- new net ~LCD_PWR_EN: R501.1, U?.4 (~SHDN)
Other:
- note added: "22V to 25.4V"
