File: pcb/usb.sch (KiCad schematic (older format))
At the start: 8 parts, among them J600 USB_B_Micro, U600 USBLC6-2SC6

Commit message: pcb: working on usb
Parts:
- removed J600: USB_B_Micro, Connector_USB:USB_Micro-B_Amphenol_10103594-0001LF_Horizontal, symbol Connector:USB_B_Micro
- removed R601: 20K, Resistor_SMD:R_0603_1608Metric, symbol Device:R
- added C? (x2): 22pF, Capacitor_SMD:C_0603_1608Metric, symbol Device:C
- added C?: 2.2uF, Capacitor_SMD:C_0603_1608Metric, symbol Device:C
- added D?: BAT54A, Package_TO_SOT_SMD:SOT-23, symbol Diode:BAT54A
- added J?: USB_A, symbol Connector:USB_A
- added R?: 27, Resistor_SMD:R_0603_1608Metric, symbol Device:R
- added R?: 10K, Resistor_SMD:R_0603_1608Metric, symbol Device:R
- added R?: 10, Resistor_SMD:R_0603_1608Metric, symbol Device:R
- added R?: 1M, Resistor_SMD:R_0603_1608Metric, symbol Device:R
- added R?: 8.06K, Resistor_SMD:R_0603_1608Metric, symbol Device:R
- added R? (x3): 0, Resistor_SMD:R_0603_1608Metric, symbol Device:R
- added U?: USB3320, Package_DFN_QFN:QFN-32-1EP_5x5mm_P0.5mm_EP3.6x3.6mm, symbol symbols:USB3320
- added Y?: 24MHz, Crystal:Crystal_SMD_3225-4Pin_3.2x2.5mm, symbol Device:Crystal_GND24
- R602: value 10K -> 1K
Connections:
- net labels added: +1V8, +3V3, +5V, PS_POR_B, USB0_CLKOUT, USB0_DATA0, USB0_DATA1, USB0_DATA2, USB0_DATA3, USB0_DATA4, USB0_DATA5, USB0_DATA6, USB0_DATA7, USB0_DIR, USB0_NXT, USB0_STP, USB_RESETB_MIO
- wire segments 32 -> 89
- no-connect marks 2 -> 4
Other:
- note added: "3.3V Regulator"
- moved on the sheet: C600, C601, D601, R600, R602, U600

Commit message: sch: working on system config
Changed lines of the file:
@@
 Date "2020-06-30"
 Rev "R0.1"
-Comp "EE300"
+Comp "Wenting Zhang"
 Comment1 "zephray@outlook.com"
 Comment2 ""
@@
 U 1 1 5C995C17
 P 7400 3200
+AR Path="/5C995C17" Ref="U600"  Part="1"
+AR Path="/5D1A413B/5C995C17" Ref="U600"  Part="1"
 F 0 "U600" H 7400 3878 50  0000 C CNN
 F 1 "USBLC6-2SC6" H 7400 3787 50  0000 C CNN
@@
 L power:GND #PWR0291
 U 1 1 5C9961F9
-P 7400 3700
-F 0 "#PWR0291" H 7400 3450 50  0001 C CNN
-F 1 "GND" H 7405 3527 50  0000 C CNN
-F 2 "" H 7400 3700 50  0001 C CNN
-F 3 "" H 7400 3700 50  0001 C CNN
-	1    7400 3700
+P 7400 3600
+F 0 "#PWR0291" H 7400 3350 50  0001 C CNN
+F 1 "GND" H 7405 3427 50  0000 C CNN
+F 2 "" H 7400 3600 50  0001 C CNN
+F 3 "" H 7400 3600 50  0001 C CNN
+	1    7400 3600
 	-1   0    0    -1
 $EndComp
@@
 Wire Wire Line
 	8600 5200 8600 5100
-NoConn ~ 7400 2700
-Wire Wire Line
-	8200 4300 8000 4300
+NoConn ~ 7400 2800
 Wire Wire Line
 	7600 4600 7600 4000
 Wire Wire Line
-	7900 3100 8000 3100
-Wire Wire Line
-	8000 3100 8000 3300
-Wire Wire Line
-	7900 3300 8000 3300
-Connection ~ 8000 3300
-Wire Wire Line
-	8000 3300 8000 4300
-Wire Wire Line
-	6900 3100 6800 3100
-Wire Wire Line
-	6800 3100 6800 3300
-Wire Wire Line
-	6900 3300 6800 3300
-Connection ~ 6800 3300
-Wire Wire Line
-	6800 3300 6800 4200
+	7800 3100 7900 3100
+Wire Wire Line
+	7900 3100 7900 3300
+Wire Wire Line
+	7800 3300 7900 3300
+Connection ~ 7900 3300
+Wire Wire Line
+	7900 3300 7900 4300
+Wire Wire Line
+	7000 3100 6900 3100
+Wire Wire Line
+	6900 3100 6900 3300
+Wire Wire Line
+	7000 3300 6900 3300
+Connection ~ 6900 3300
+Wire Wire Line
+	6900 3300 6900 4200
 Wire Wire Line
 	6500 2900 6500 3000
@@
 USB_DP
 Wire Wire Line
-	8200 4200 6800 4200
-Wire Wire Line
-	6800 4200 6700 4200
+	8200 4200 6900 4200
 Wire Wire Line
 	6700 4200 6700 4800
 Wire Wire Line
 	6700 4800 5600 4800
-Connection ~ 6800 4200
 Wire Wire Line
 	5600 4900 6800 4900
@@
 	6800 4900 6800 4300
 Wire Wire Line
-	6800 4300 8000 4300
-Connection ~ 8000 4300
+	6800 4300 7900 4300
 Text GLabel 4300 3100 0    50   BiDi ~ 0
 USB0_DATA7
@@
 	6100 3100 6100 3000
 NoConn ~ 5600 3400
+Connection ~ 7900 4300
+Wire Wire Line
+	7900 4300 8200 4300
+Connection ~ 6900 4200
+Wire Wire Line
+	6700 4200 6900 4200
 $EndSCHEMATC
